Commit message: Add files via upload

File: urdf/catvehicle.xacro (robot description, xacro)
@@ -178,5 +178,5 @@
     <joint name="inertial_joint" type="fixed">
         <parent link="base_link"/>
-        <child link="main_mass"/>
+        <child link="main_mass"/> <!-- previously main_mass -->
         <origin xyz="0 0 0" rpy="0 0 0"/>
     </joint>
